File: scatter42/scatter42.kicad_pcb (KiCad board)
At the start: 2 copper layers, 267 x 102.7 mm, 112 parts, among them J0 MJ-4PP-9, J1 MJ-4PP-9, SW0 SW_PUSH, SW1 SW_PUSH, SW10 SW_PUSH, SW11 SW_PUSH, SW12 SW_PUSH, SW13 SW_PUSH, SW14 SW_PUSH, SW15 SW_PUSH, SW16 SW_PUSH, SW17 SW_PUSH, SW18 SW_PUSH, SW19 SW_PUSH, SW2 SW_PUSH, SW20 SW_PUSH, SW21 SW_PUSH, SW22 SW_PUSH, SW23 SW_PUSH, SW24 SW_PUSH, SW25 SW_PUSH, SW26 SW_PUSH, SW27 SW_PUSH, SW28 SW_PUSH, SW29 SW_PUSH, SW3 SW_PUSH, SW30 SW_PUSH, SW31 SW_PUSH, SW32 SW_PUSH, SW33 SW_PUSH, SW34 SW_PUSH, SW35 SW_PUSH, SW36 SW_PUSH, SW37 SW_PUSH, SW38 SW_PUSH, SW39 SW_PUSH, SW4 SW_PUSH, SW40 SW_PUSH, SW41 SW_PUSH, SW5 SW_PUSH, SW6 SW_PUSH, SW7 SW_PUSH, SW8 SW_PUSH, SW9 SW_PUSH, U0 ProMicro, U1 ProMicro

Commit message: for v1.1.0
Parts:
- removed CUT0, CUT1, CUT10, CUT11, CUT2, CUT3, CUT4, CUT5, CUT6, CUT7, CUT8, CUT9: Val**, foostan_kbd:IM_HOLE
- added HOLE10: HOLE10, foostan_kbd:IM_HOLE, F.Cu at (139.1, 50.9)
- added HOLE11: HOLE11, foostan_kbd:IM_HOLE, F.Cu at (139.1, 51.9)
- added HOLE12: HOLE12, foostan_kbd:IM_HOLE, F.Cu at (139.1, 52.9)
- added HOLE13: HOLE13, foostan_kbd:IM_HOLE, F.Cu at (139.1, 53.9)
- added HOLE14: HOLE14, foostan_kbd:IM_HOLE, F.Cu at (139.1, 54.9)
- added HOLE15: HOLE15, foostan_kbd:IM_HOLE, F.Cu at (139.1, 56.0)
- added HOLE16: HOLE16, foostan_kbd:IM_HOLE, F.Cu at (158.2, 50.9)
- added HOLE17: HOLE17, foostan_kbd:IM_HOLE, F.Cu at (158.2, 51.9)
- added HOLE18: HOLE18, foostan_kbd:IM_HOLE, F.Cu at (158.2, 52.9)
- added HOLE19: HOLE19, foostan_kbd:IM_HOLE, F.Cu at (158.2, 53.9)
- added HOLE20: HOLE20, foostan_kbd:IM_HOLE, F.Cu at (158.2, 55.0)
- added HOLE21: HOLE21, foostan_kbd:IM_HOLE, F.Cu at (158.2, 56.0)
- D21, D22, D23, D24, D25, D26, D27, D28, D29, D30, D31, D32, D33, D34, D35, D36, D37, D38, D39, D40, D41, J1, RSW1, SW21, SW22, SW23, SW24, SW25, SW26, SW27, SW28, SW29, SW30, SW31, SW32, SW33, SW34, SW35, SW36, SW37, SW38, SW39, SW40, SW41, U1: moved to B.Cu
- moved D41 86.0 mm to (162.1, 25.7), turned to 330 degrees
- moved SW23 85.8 mm to (229.0, 111.5)
- moved SW22 76.3 mm to (248.1, 106.7)
- moved SW24 76.2 mm to (210.0, 106.7)
- moved SW41 75.0 mm to (158.8, 31.2), turned to 330 degrees
- moved D23 73.5 mm to (229.0, 105.4)
- moved D40 70.1 mm to (180.6, 33.8), turned to 345 degrees
- moved SW25 66.8 mm to (191.0, 102.0)
- moved SW21 66.7 mm to (267.2, 102.0)
- moved HOLE9 65.4 mm to (168.9, 35.9)
- moved D39 65.2 mm to (200.5, 36.2)
- moved D24 63.8 mm to (210.1, 100.5)
- moved D22 63.8 mm to (248.2, 100.5)
- moved D36 60.5 mm to (267.2, 38.6)
- moved SW40 58.4 mm to (178.9, 39.6), turned to 345 degrees
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Routing:
- net row3_r: track 230.0 -> 286.6 mm, vias 4 -> 1
- net row2: track 187.1 -> 242.9 mm, vias 4 -> 1
- net row2_r: track 153.8 -> 194.2 mm, vias 5 -> 2
- net col4: track 145.0 -> 104.6 mm
- net row3: track 281.5 -> 311.5 mm, vias 3 -> 1
- net col1_r: track 140.8 -> 170.7 mm, vias 1 -> 0
- net row1_r: track 147.1 -> 170.3 mm, vias 4 -> 2
- net Net-(D41-Pad2): track 36.0 -> 15.3 mm, vias 2 -> 1
- net GND: track 74.5 -> 58.3 mm
- net col2: track 122.4 -> 138.4 mm, vias 1 -> 0
- net col3_r: track 110.6 -> 126.4 mm, vias 1 -> 0
- net col1: track 157.4 -> 144.3 mm
- net col5_r: track 69.9 -> 57.4 mm, vias 1 -> 0
- net col2_r: track 131.3 -> 142.1 mm, vias 1 -> 0
- net VDD: track 44.9 -> 35.4 mm, vias 1 -> 0
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- removed copper zone on B.Cu, net GND
- removed copper zone on F.Cu, net GND
- removed copper zone on B.Cu, net GNDA
- removed copper zone on F.Cu, net GNDA
Other:
- board size 267 x 102.7 mm -> 260.1 x 107.6 mm
- board text added: "Scatter42 v1.1.0: PCB designed by @bbrfkr"
- board text removed: "Scatter42 v1.0.0 Designed by bbrfkr"

Commit message: fill gnd and gnda
Routing:
- added copper zone on B.Cu, net GND
- added copper zone on F.Cu, net GND
- added copper zone on B.Cu, net GNDA
- added copper zone on F.Cu, net GNDA
Changed lines of the file:
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@@
       (outputformat 1)
       (mirror false)
-      (drillshape 1)
+      (drillshape 0)
       (scaleselection 1)
       (outputdirectory ""))
@@
   (segment (start 161.1433 80.7661) (end 162.3684 81.9912) (width 0.25) (layer F.Cu) (net 72))
   (segment (start 151.3692 29.8611) (end 150.3671 31.5967) (width 0.25) (layer F.Cu) (net 72))
+  (zone (net 57) (net_name GNDA) (layer F.Cu) (hatch edge 0.508)
+    (connect_pads (clearance 0.508))
+    (min_thickness 0.254)
+    (fill yes (arc_segments 32) (thermal_gap 0.508) (thermal_bridge_width 0.508))
+    (polygon
+      (pts
+        (xy 282.0543 29.0322) (xy 282.7147 127) (xy 155.8544 129.6543) (xy 156.5148 128.651) (xy 156.1846 47.2948)
+        (xy 141.9098 35.6743) (xy 154.1907 14.4145)
+      )
+    )
+  )
+  (zone (net 57) (net_name GNDA) (layer B.Cu) (hatch edge 0.508)
+    (connect_pads (clearance 0.508))
+    (min_thickness 0.254)
+    (fill yes (arc_segments 32) (thermal_gap 0.508) (thermal_bridge_width 0.508))
+    (polygon
+      (pts
+        (xy 282.061999 28.946013) (xy 282.722399 126.913813) (xy 155.862099 129.568113) (xy 156.522499 128.564813) (xy 156.192299 47.208613)
+        (xy 141.917499 35.588113) (xy 154.198399 14.328313)
+      )
+    )
+  )
+  (zone (net 54) (net_name GND) (layer F.Cu) (hatch edge 0.508)
+    (connect_pads (clearance 0.508))
+    (min_thickness 0.254)
+    (fill yes (arc_segments 32) (thermal_gap 0.508) (thermal_bridge_width 0.508))
+    (polygon
+      (pts
+        (xy 139.319 93.3704) (xy 155.2575 103.3399) (xy 144.1069 125.6538) (xy 15.7861 111.3028) (xy 15.7861 15.6718)
+        (xy 140.5128 14.4653)
+      )
+    )
+  )
+  (zone (net 54) (net_name GND) (layer B.Cu) (hatch edge 0.508)
+    (connect_pads (clearance 0.508))
+    (min_thickness 0.254)
+    (fill yes (arc_segments 32) (thermal_gap 0.508) (thermal_bridge_width 0.508))
+    (polygon
+      (pts
+        (xy 139.351043 93.528316) (xy 155.289543 103.497816) (xy 144.138943 125.811716) (xy 15.818143 111.460716) (xy 15.818143 15.829716)
+        (xy 140.544843 14.623216)
+      )
+    )
+  )
 )

Commit message: mod cutline and silk
Routing:
- net row3: track 311.5 -> 188.3 mm, vias 1 -> 0
- net row3_r: track 286.6 -> 175.1 mm, vias 1 -> 0
- net col1_r: track 170.7 -> 238.7 mm, vias 0 -> 2
- net row2: track 242.9 -> 176.0 mm
- net col1: track 144.3 -> 209.1 mm, vias 1 -> 0
- net row1_r: track 170.3 -> 120.4 mm, vias 2 -> 1
- net row0_r: track 164.7 -> 121.5 mm, vias 2 -> 0
- net row2_r: track 194.2 -> 152.2 mm, vias 2 -> 0
- net row1: track 167.6 -> 142.9 mm, vias 3 -> 2
- net col3: track 130.0 -> 111.3 mm
- net col2_r: track 142.1 -> 129.8 mm
- net col0_r: track 180.4 -> 192.4 mm
- net row0: track 167.5 -> 179.3 mm, vias 3 -> 0
- net col2: track 138.4 -> 129.8 mm, vias 0 -> 1
- net col3_r: track 126.4 -> 118.8 mm, vias 0 -> 2
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Other:
- outline, holes or cut-outs redrawn
- board text added: "Scatter42 v1.1.1: PCB designed by @bbrfkr"
- board text removed: "Scatter42 v1.1.0: PCB designed by @bbrfkr"

Commit message: paste logo to pcb
Parts:
- added G***: LOGO, bbrfkr_logos:logo, B.Cu at (227.2, 37.8)
- added G***: LOGO, bbrfkr_logos:logo, F.Cu at (227.2, 37.8)
- added G***: LOGO, bbrfkr_logos:logo, B.Cu at (70.5, 101.6)
- added G***: LOGO, bbrfkr_logos:logo, F.Cu at (70.5, 101.6)
Other:
- board text added: "Scatter42 v1.1.2: PCB designed by @bbrfkr"
- board text removed: "Scatter42 v1.1.1: PCB designed by @bbrfkr"

Commit message: mod for scatter42
Parts:
- added CASE00: CASE00, bbrfkr_kbd:statter42-plate, F.Cu at (86.2, 69.9)
- added CASE01: CASE01, bbrfkr_kbd:statter42-plate, F.Cu at (211.0, 69.4)
- added HOLE22: HOLE22, foostan_kbd:HOLE, F.Cu at (121.9, 70.2)
- added HOLE23: HOLE23, foostan_kbd:HOLE, F.Cu at (134.7, 70.2)
- added HOLE24: HOLE24, foostan_kbd:HOLE, F.Cu at (162.6, 69.2)
- added HOLE25: HOLE25, foostan_kbd:HOLE, F.Cu at (175.3, 69.2)
- LOGO00: renamed from G***; value LOGO -> LOGO00; footprint bbrfkr_logos:logo -> bbrfkr_kbd:scatter42-logo
- LOGO01: renamed from G***; value LOGO -> LOGO01; footprint bbrfkr_logos:logo -> bbrfkr_kbd:scatter42-logo
- LOGO02: renamed from G***; value LOGO -> LOGO02; footprint bbrfkr_logos:logo -> bbrfkr_kbd:scatter42-logo
- LOGO03: renamed from G***; value LOGO -> LOGO03; footprint bbrfkr_logos:logo -> bbrfkr_kbd:scatter42-logo
- moved HOLE10 16.0 mm to (139.2, 66.8)
- moved HOLE14 16.0 mm to (139.2, 70.9)
- moved HOLE11 16.0 mm to (139.2, 67.8)
- moved HOLE12 16.0 mm to (139.2, 68.8)
- moved HOLE13 16.0 mm to (139.2, 69.8)
- moved HOLE15 16.0 mm to (139.2, 71.9)
- moved HOLE17 15.9 mm to (158.1, 67.8)
- moved HOLE19 15.9 mm to (158.1, 69.8)
- moved HOLE21 15.9 mm to (158.1, 71.9)
- moved HOLE16 15.9 mm to (158.1, 66.8)
- moved HOLE18 15.9 mm to (158.1, 68.8)
- moved HOLE20 15.9 mm to (158.1, 70.9)
- moved J0 8.11 mm to (137.5, 82.9)
- moved RSW0 8.11 mm to (132.9, 76.7)
- moved J1 7.98 mm to (159.7, 56.6)
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Routing:
- net row0: track 179.3 -> 141.3 mm, vias 0 -> 3
- net row2: track 176.0 -> 208.2 mm, vias 1 -> 0
- net col1_r: track 238.7 -> 270.8 mm, vias 2 -> 0
- net row1_r: track 120.4 -> 141.6 mm
- net row2_r: track 152.2 -> 132.0 mm, vias 0 -> 1
- net row1: track 142.9 -> 124.8 mm
- net reset: track 36.8 -> 51.8 mm
- net GNDA: track 59.3 -> 72.0 mm
- net col2: track 129.8 -> 142.1 mm, vias 1 -> 0
- net col3: track 111.3 -> 121.9 mm
- net data: track 42.1 -> 52.2 mm
- net col4: track 111.7 -> 102.1 mm, vias 0 -> 1
- net reset_r: track 31.9 -> 40.8 mm
- net col1: track 209.1 -> 200.4 mm
- net VCC: track 37.6 -> 45.8 mm
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Other:
- board size 260.1 x 107.6 mm -> 260 x 107.6 mm
- board text added: "Scatter42 v1.1.3: PCB designed by @bbrfkr"
- board text removed: "Scatter42 v1.1.2: PCB designed by @bbrfkr"

Commit message: mod to allow to use kailh choc switch
Parts:
- CASE00, CASE01: footprint bbrfkr_kbd:statter42-plate -> scatter42:statter42-plate
- D0, D1, D10, D11, D12, D13, D14, D15, D16, D17, D18, D19, D2, D20, D21, D22, D23, D24, D25, D26, D27, D28, D29, D3, D30, D31, D32, D33, D34, D35, D36, D37, D38, D39, D4, D40, D41, D5, D6, D7, D8, D9: footprint foostan_kbd:D3_SMD -> scatter42:D3_SMD
- HOLE0, HOLE1, HOLE2, HOLE3, HOLE4, HOLE5, HOLE6, HOLE7, HOLE8, HOLE9: footprint foostan_kbd:HOLE -> scatter42:HOLE
- HOLE22, HOLE23, HOLE24, HOLE25: footprint foostan_kbd:HOLE -> scatter42:M2_Hole_TH
- J0, J1: footprint foostan_kbd:MJ-4PP-9_1side -> scatter42:MJ-4PP-9_1side
- LOGO00, LOGO01, LOGO02, LOGO03: footprint bbrfkr_kbd:scatter42-logo -> scatter42:scatter42-logo
- RSW0, RSW1: footprint foostan_kbd:ResetSW -> scatter42:ResetSW
- SW0, SW1, SW10, SW11, SW12, SW13, SW14, SW15, SW16, SW17, SW18, SW19, SW2, SW20, SW21, SW22, SW23, SW24, SW25, SW26, SW27, SW28, SW29, SW3, SW30, SW31, SW32, SW33, SW34, SW35, SW36, SW37, SW38, SW39, SW4, SW40, SW41, SW5, SW6, SW7, SW8, SW9: footprint foostan_kbd:CherryMX_Hotswap -> scatter42:CherryMX_Choc_Hotswap
- U0, U1: footprint foostan_kbd:ProMicro_v3 -> scatter42:ProMicro_v3
- moved D41 6.72 mm to (166.6, 30.6), turned to 60 degrees
- moved D36 6.67 mm to (273.5, 40.6), turned to 90 degrees
- moved D33 6.65 mm to (235.4, 69.1), turned to 90 degrees
- moved D31 6.61 mm to (273.5, 59.7), turned to 90 degrees
- moved D37 6.60 mm to (254.4, 45.4), turned to 90 degrees
- moved D23 6.59 mm to (235.3, 107.3), turned to 90 degrees
- moved D38 6.58 mm to (235.4, 50.1), turned to 90 degrees
- moved D0 6.58 mm to (36.3, 41.5), turned to 90 degrees
- moved D29 6.57 mm to (216.3, 83.4), turned to 90 degrees
- moved D28 6.57 mm to (235.3, 88.3), turned to 90 degrees
- moved D1 6.56 mm to (55.4, 36.8), turned to 90 degrees
- moved D18 6.55 mm to (103.0, 101.0), turned to 90 degrees
- moved D9 6.55 mm to (112.6, 60.5), turned to 90 degrees
- moved D24 6.54 mm to (216.3, 102.5), turned to 90 degrees
- moved D34 6.54 mm to (216.3, 64.3), turned to 90 degrees
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Routing:
- net col1_r: track 270.8 -> 149.3 mm, vias 0 -> 2
- net row2: track 208.2 -> 166.5 mm
- net col4: track 102.1 -> 139.7 mm
- net row0_r: track 122.9 -> 156.1 mm, vias 0 -> 1
- net row0: track 141.3 -> 173.0 mm, vias 3 -> 0
- net row3_r: track 174.6 -> 194.9 mm, vias 0 -> 2
- net col0_r: track 193.6 -> 209.2 mm, vias 0 -> 4
- net col3: track 121.9 -> 136.5 mm, vias 0 -> 2
- net data_r: track 56.2 -> 70.5 mm
- net VCC: track 45.8 -> 59.5 mm
- net col4_r: track 111.0 -> 123.3 mm
- net row3: track 191.0 -> 180.6 mm, vias 0 -> 1
- net col5: track 50.7 -> 61.1 mm, vias 0 -> 1
- net Net-(D35-Pad2): track 13.0 -> 22.9 mm
- net row1: track 124.8 -> 116.5 mm, vias 2 -> 0
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Other:
- board text added: "Scatter42 v1.2.0: PCB designed by @bbrfkr"
- board text removed: "Scatter42 v1.1.3: PCB designed by @bbrfkr"

Commit message: mod for v1.3.0
Parts:
- removed CASE00: CASE00, scatter42:statter42-plate
- removed CASE01: CASE01, scatter42:statter42-plate
- removed HOLE14: HOLE14, foostan_kbd:IM_HOLE
- removed HOLE15: HOLE15, foostan_kbd:IM_HOLE
- removed HOLE16: HOLE16, foostan_kbd:IM_HOLE
- removed HOLE17: HOLE17, foostan_kbd:IM_HOLE
- removed HOLE18: HOLE18, foostan_kbd:IM_HOLE
- removed HOLE19: HOLE19, foostan_kbd:IM_HOLE
- removed HOLE20: HOLE20, foostan_kbd:IM_HOLE
- removed HOLE21: HOLE21, foostan_kbd:IM_HOLE
- removed HOLE22: HOLE22, scatter42:M2_Hole_TH
- removed HOLE23: HOLE23, scatter42:M2_Hole_TH
- removed HOLE24: HOLE24, scatter42:M2_Hole_TH
- removed HOLE25: HOLE25, scatter42:M2_Hole_TH
- removed LOGO00: LOGO00, scatter42:scatter42-logo
- removed LOGO01: LOGO01, scatter42:scatter42-logo
- removed LOGO02: LOGO02, scatter42:scatter42-logo
- removed LOGO03: LOGO03, scatter42:scatter42-logo
- added G***: LOGO, scatter42:scatter42-logo, F.Cu at (296.6, 182.5)
- added G***: LOGO, scatter42:scatter42-logo, B.Cu at (296.6, 182.5)
- added G***: LOGO, scatter42:scatter42-logo, B.Cu at (123.1, 182.5)
- added G***: LOGO, scatter42:scatter42-logo, F.Cu at (123.1, 182.5)
- added LED0: SK6812MINI, scatter42:SK6812MINI_underglow_rev, F.Cu at (144.8, 105.7)
- added LED1: SK6812MINI, scatter42:SK6812MINI_underglow_rev, F.Cu at (81.2, 110.4)
- added LED2: SK6812MINI, scatter42:SK6812MINI_underglow_rev, F.Cu at (93.7, 176.6)
- added LED3: SK6812MINI, scatter42:SK6812MINI_underglow_rev, F.Cu at (126.1, 162.3)
- added LED4: SK6812MINI, scatter42:SK6812MINI_underglow_rev, F.Cu at (162.5, 179.5)
- added LED5: SK6812MINI, scatter42:SK6812MINI_underglow_rev, F.Cu at (274.1, 105.6)
- added LED6: SK6812MINI, scatter42:SK6812MINI_underglow_rev, F.Cu at (337.9, 110.4)
- added LED7: SK6812MINI, scatter42:SK6812MINI_underglow_rev, F.Cu at (325.4, 176.6)
- added LED8: SK6812MINI, scatter42:SK6812MINI_underglow_rev, F.Cu at (292.8, 162.3)
- added LED9: SK6812MINI, scatter42:SK6812MINI_underglow_rev, F.Cu at (256.6, 179.5)
- added OL0: OLED, scatter42:OLED_v2, F.Cu at (172.5, 142.4)
- added OL1: OLED, scatter42:OLED_v2, F.Cu at (246.7, 142.4)
- D21, D22, D23, D24, D25, D26, D27, D28, D29, D30, D31, D32, D33, D34, D35, D36, D37, D38, D39, D40, D41, J1, RSW1, SW21, SW22, SW23, SW24, SW25, SW26, SW27, SW28, SW29, SW30, SW31, SW32, SW33, SW34, SW35, SW36, SW37, SW38, SW39, SW40, SW41, U1: moved to F.Cu
- HOLE10, HOLE11: footprint foostan_kbd:IM_HOLE -> scatter42:HOLE
- HOLE12, HOLE13: footprint foostan_kbd:IM_HOLE -> scatter42:M2_Hole_TH
- HOLE5, HOLE6: footprint scatter42:HOLE -> scatter42:M2_Hole_TH
- moved HOLE9 216.0 mm to (331.8, 178.5)
- moved HOLE10 178.2 mm to (286.8, 166.6)
- moved SW41 177.6 mm to (226.7, 195.5), turned to 45 degrees
- moved D41 176.8 mm to (234.2, 194.1), turned to 315 degrees
- moved D40 161.9 mm to (253.2, 184.5), turned to 290 degrees
- moved D36 161.6 mm to (350.2, 182.8), turned to 270 degrees
- moved D39 159.5 mm to (274.0, 182.8), turned to 270 degrees
- moved SW40 157.8 mm to (245.9, 182.7), turned to 20 degrees
- moved SW36 154.2 mm to (344.0, 178.5)
- moved HOLE11 153.1 mm to (235.0, 187.2)
- moved SW39 151.8 mm to (267.8, 178.5)
- moved D37 145.1 mm to (331.2, 168.5), turned to 270 degrees
- moved HOLE8 142.0 mm to (343.9, 107.1)
- moved HOLE13 139.8 mm to (252.6, 151.6)
- moved SW37 138.0 mm to (324.9, 164.3)
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Connections:
- U0 pad 1: Net-(U0-Pad1) -> LED
- U0 pad 5: Net-(U0-Pad5) -> SDA
- U0 pad 6: Net-(U0-Pad6) -> SCL
- U1 pad 1: Net-(U1-Pad1) -> LED_r
- U1 pad 5: Net-(U1-Pad5) -> SDA_r
- U1 pad 6: Net-(U1-Pad6) -> SCL_r
Routing:
- net GNDA: track 73.5 -> 303.0 mm, vias 0 -> 1
- net VDD: track 42.1 -> 269.7 mm, vias 0 -> 3
- net GND: track 68.1 -> 287.2 mm, vias 0 -> 2
- net VCC: track 59.5 -> 259.7 mm, vias 0 -> 2
- net Net-(LED1-Pad1): track 0.00 -> 107.9 mm
- net Net-(LED5-Pad1): track 0.00 -> 80.5 mm
- net Net-(LED0-Pad1): track 0.00 -> 73.3 mm
- net Net-(LED6-Pad1): track 0.00 -> 69.4 mm
- net row3_r: track 194.9 -> 255.8 mm
- net row3: track 180.6 -> 232.7 mm, vias 1 -> 0
- net row2_r: track 128.9 -> 180.7 mm, vias 4 -> 3
- net Net-(LED3-Pad1): track 0.00 -> 48.8 mm, vias 0 -> 2
- net Net-(LED2-Pad1): track 0.00 -> 44.2 mm
- net col0_r: track 209.2 -> 167.4 mm, vias 4 -> 1
- net Net-(LED8-Pad1): track 0.00 -> 39.7 mm
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Other:
- board size 260 x 107.6 mm -> 290.8 x 120.1 mm
- board text added: "Scatter42 v1.3.0 PCB designed by @bbrfkr"
- board text removed: "Scatter42 v1.2.0: PCB designed by @bbrfkr"
