File: scatter42/scatter42.sch (KiCad schematic (older format))
At the start: 90 parts, among them J0 MJ-4PP-9, J1 MJ-4PP-9, SW0 SW_PUSH, SW1 SW_PUSH, SW10 SW_PUSH, SW11 SW_PUSH, SW12 SW_PUSH, SW13 SW_PUSH, SW14 SW_PUSH, SW15 SW_PUSH, SW16 SW_PUSH, SW17 SW_PUSH, SW18 SW_PUSH, SW19 SW_PUSH, SW2 SW_PUSH, SW20 SW_PUSH, SW21 SW_PUSH, SW22 SW_PUSH, SW23 SW_PUSH, SW24 SW_PUSH, SW25 SW_PUSH, SW26 SW_PUSH, SW27 SW_PUSH, SW28 SW_PUSH, SW29 SW_PUSH, SW3 SW_PUSH, SW30 SW_PUSH, SW31 SW_PUSH, SW32 SW_PUSH, SW33 SW_PUSH, SW34 SW_PUSH, SW35 SW_PUSH, SW36 SW_PUSH, SW37 SW_PUSH, SW38 SW_PUSH, SW39 SW_PUSH, SW4 SW_PUSH, SW40 SW_PUSH, SW41 SW_PUSH, SW5 SW_PUSH, SW6 SW_PUSH, SW7 SW_PUSH, SW8 SW_PUSH, SW9 SW_PUSH, U0 ProMicro, U1 ProMicro

Commit message: mod cutline and silk
Parts:
- J0, J1: footprint foostan_kbd:MJ-4PP-9 -> foostan_kbd:MJ-4PP-9_1side
Changed lines of the file:
@@
 F 0 "J0" H 881 2726 50  0000 C CNN
 F 1 "MJ-4PP-9" H 881 2635 50  0000 C CNN
-F 2 "foostan_kbd:MJ-4PP-9" H 1125 2625 50  0001 C CNN
+F 2 "foostan_kbd:MJ-4PP-9_1side" H 1125 2625 50  0001 C CNN
 F 3 "~" H 1125 2625 50  0001 C CNN
 	1    850  2450
@@
 F 0 "J1" H 8431 2726 50  0000 C CNN
 F 1 "MJ-4PP-9" H 8431 2635 50  0000 C CNN
-F 2 "foostan_kbd:MJ-4PP-9" H 8675 2625 50  0001 C CNN
+F 2 "foostan_kbd:MJ-4PP-9_1side" H 8675 2625 50  0001 C CNN
 F 3 "~" H 8675 2625 50  0001 C CNN
 	1    8400 2450

Commit message: mod to allow to use kailh choc switch
Parts:
- D0, D1, D10, D11, D12, D13, D14, D15, D16, D17, D18, D19, D2, D20, D21, D22, D23, D24, D25, D26, D27, D28, D29, D3, D30, D31, D32, D33, D34, D35, D36, D37, D38, D39, D4, D40, D41, D5, D6, D7, D8, D9: footprint foostan_kbd:D3_SMD -> scatter42:D3_SMD
- J0, J1: footprint foostan_kbd:MJ-4PP-9_1side -> scatter42:MJ-4PP-9_1side
- RSW0, RSW1: footprint foostan_kbd:ResetSW -> scatter42:ResetSW
- SW0, SW1, SW10, SW11, SW12, SW13, SW14, SW15, SW16, SW17, SW18, SW19, SW2, SW20, SW21, SW22, SW23, SW24, SW25, SW26, SW27, SW28, SW29, SW3, SW30, SW31, SW32, SW33, SW34, SW35, SW36, SW37, SW38, SW39, SW4, SW40, SW41, SW5, SW6, SW7, SW8, SW9: footprint foostan_kbd:CherryMX_Hotswap -> scatter42:CherryMX_Choc_Hotswap
- U0, U1: footprint foostan_kbd:ProMicro_v3 -> scatter42:ProMicro_v3

Commit message: mod for v1.3.0
Parts:
- added LED0, LED1, LED2, LED3, LED4, LED5, LED6, LED7, LED8, LED9: SK6812MINI, scatter42:SK6812MINI_underglow_rev, symbol scatter42:SK6812MINI
- added OL0, OL1: OLED, scatter42:OLED_v2, symbol scatter42:OLED
- J0, J1: symbol foostan_kbd:MJ-4PP-9 -> scatter42:MJ-4PP-9
- RSW0, RSW1, SW0, SW1, SW10, SW11, SW12, SW13, SW14, SW15, SW16, SW17, SW18, SW19, SW2, SW20, SW21, SW22, SW23, SW24, SW25, SW26, SW27, SW28, SW29, SW3, SW30, SW31, SW32, SW33, SW34, SW35, SW36, SW37, SW38, SW39, SW4, SW40, SW41, SW5, SW6, SW7, SW8, SW9: symbol foostan_kbd:SW_PUSH -> scatter42:SW_PUSH
- U0, U1: symbol foostan_kbd:ProMicro -> scatter42:ProMicro
Connections:
- net labels added: LED, LED_r, SCL, SCL_r, SDA, SDA_r
- wire segments 106 -> 180
- no-connect marks 18 -> 14
