File: molecule_v2_plate/molecule_v2_plate.kicad_pcb (KiCad board)
At the start: 2 copper layers, 282.6 x 134.6 mm, 0 parts

Commit message: wip
Routing:
- removed copper zone on B.Cu, net (none)
- removed copper zone on F.Cu, net (none)
Other:
- board size 282.6 x 134.6 mm -> 281.4 x 133.8 mm
