File: molecule_v2/molecule_v2.kicad_pcb (KiCad board)
At the start: 2 copper layers, 282 x 132.8 mm, 161 parts, among them J0 USB_C_Receptacle_USB2.0, SW0 SW_PUSH, SW1 SW_PUSH, SW10 SW_PUSH, SW11 SW_PUSH, SW12 SW_PUSH, SW13 SW_PUSH, SW14 SW_PUSH, SW15 SW_PUSH, SW16 SW_PUSH, SW17 SW_PUSH, SW18 SW_PUSH, SW19 SW_PUSH, SW2 SW_PUSH, SW20 SW_PUSH, SW21 SW_PUSH, SW22 SW_PUSH, SW23 SW_PUSH, SW24 SW_PUSH, SW25 SW_PUSH, SW26 SW_PUSH, SW27 SW_PUSH, SW28 SW_PUSH, SW29 SW_PUSH, SW3 SW_PUSH, SW30 SW_PUSH, SW31 SW_PUSH, SW32 SW_PUSH, SW33 SW_PUSH, SW34 SW_PUSH, SW35 SW_PUSH, SW36 SW_PUSH, SW37 SW_PUSH, SW38 SW_PUSH, SW39 SW_PUSH, SW4 SW_PUSH, SW5 SW_PUSH, SW6 SW_PUSH, SW7 SW_PUSH, SW8 SW_PUSH, SW9 SW_PUSH, U0 ATmega32U4-AU, U1 PMW3360DM-T2QU, U2 TLV70019DDCR, U3 74LVC1T45GW,125, U4 74LVC1T45GW,125, U5 74LVC1T45GW,125, U6 74LVC1T45GW,125, U7 74LVC1T45GW,125, Y0 16Mhz

Commit message: wip
Parts:
- moved C1 41.5 mm to (189.7, 109.6)
- moved C2 41.5 mm to (193.5, 109.6)
- moved C3 41.5 mm to (197.5, 109.7)
- moved C4 41.5 mm to (201.4, 109.7)
- moved R7 27.9 mm to (233.8, 90.8), turned to 270 degrees
- moved Y0 27.4 mm to (205.7, 109.6)
- moved C0 27.1 mm to (219.5, 118.7), turned to 0 degrees
- moved U3 25.4 mm to (222.6, 124.6), turned to 180 degrees
- moved U7 14.5 mm to (222.7, 129.0)
- moved R5 11.1 mm to (232.9, 137.0)
- moved C10 10.4 mm to (199.4, 136.7)
- moved C9 10.4 mm to (199.5, 140.5)
- moved C5 8.42 mm to (230.9, 90.8)
- moved R4 7.70 mm to (236.7, 90.8)
- moved R6 7.30 mm to (227.2, 123.1)
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Connections:
- U0 pad 18: col0 -> row2
- U0 pad 19: col1 -> row1
- U0 pad 22: col3 -> row0
- U0 pad 25: col2 -> col4
- U0 pad 26: col4 -> col3
- U0 pad 27: col5 -> col2
- U0 pad 28: row0 -> col1
- U0 pad 29: row1 -> col0
- U0 pad 30: row2 -> Net-(U0-Pad30)
- U0 pad 37: Net-(U0-Pad37) -> col9
- U0 pad 38: col9 -> col8
- U0 pad 39: col8 -> col7
- U0 pad 40: col7 -> col6
- U0 pad 41: col6 -> col5
Routing:
- net GND: track 1666.3 -> 0.00 mm, vias 59 -> 0
- net VCC: track 1501.9 -> 0.00 mm, vias 11 -> 0
- net row2: track 409.9 -> 0.00 mm, vias 18 -> 0
- net row3: track 404.2 -> 0.00 mm, vias 14 -> 0
- net row1: track 398.4 -> 0.00 mm, vias 19 -> 0
- net row0: track 355.3 -> 0.00 mm, vias 19 -> 0
- net LED: track 300.9 -> 0.00 mm, vias 2 -> 0
- net col7: track 271.9 -> 0.00 mm, vias 8 -> 0
- net col2: track 224.8 -> 0.00 mm, vias 10 -> 0
- net col0: track 215.4 -> 0.00 mm, vias 4 -> 0
- net col9: track 204.5 -> 0.00 mm, vias 10 -> 0
- net col6: track 200.1 -> 0.00 mm, vias 6 -> 0
- net col1: track 196.6 -> 0.00 mm, vias 8 -> 0
- net col3: track 189.9 -> 0.00 mm, vias 10 -> 0
- net col8: track 180.6 -> 0.00 mm, vias 10 -> 0
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- removed copper zone on B.Cu, net (none)
- removed copper zone on F.Cu, net (none)
Other:
- board size 282 x 132.8 mm -> 17.9 x 17.9 mm

Commit message: wip
Parts:
- removed D40, D41, D42, D43, D44, D45: WS2812B, LED_SMD:LED_WS2812B_PLCC4_5.0x5.0mm_P3.2mm
- added R8: 10k, Resistor_SMD:R_1206_3216Metric, B.Cu at (201.5, 147.0)
- C7: value 0.1μF -> 4.7μF
- C8: value 4.7μF -> 0.1μF
- RESET_SW0: value SW_PUSH -> TS-1187A-B-A-B; footprint Keebio-Parts:SW_Tactile_SPST_Angled_MJTP1117 -> TS-1187A-B-A-B:SW_TS-1187A-B-A-B; moved to F.Cu
- moved RESET_SW0 30.3 mm to (234.8, 107.7), turned to 0 degrees
Connections:
- C9 pad 1: VCC -> VDD
- LED0 pad 4: Net-(D40-Pad2) -> LED
- R5 pad 1: VCC -> VDD
- R6 pad 1: VCC -> VDD
- U1 pad 4: VCC -> VDD
- U1 pad 5: VCC -> VDD
- U2 pad 5: VCC -> VDD
- U3 pad 6: VCC -> VDD
- U4 pad 6: VCC -> VDD
- U5 pad 6: VCC -> VDD
- U6 pad 6: VCC -> VDD
- U7 pad 6: VCC -> VDD
Other:
- board size 17.9 x 17.9 mm -> 19.4 x 19.4 mm
