File: molecule_v2/molecule_v2.sch (KiCad schematic (older format))
At the start: 157 parts, among them J0 USB_C_Receptacle_USB2.0, SW0 SW_PUSH, SW1 SW_PUSH, SW10 SW_PUSH, SW11 SW_PUSH, SW12 SW_PUSH, SW13 SW_PUSH, SW14 SW_PUSH, SW15 SW_PUSH, SW16 SW_PUSH, SW17 SW_PUSH, SW18 SW_PUSH, SW19 SW_PUSH, SW2 SW_PUSH, SW20 SW_PUSH, SW21 SW_PUSH, SW22 SW_PUSH, SW23 SW_PUSH, SW24 SW_PUSH, SW25 SW_PUSH, SW26 SW_PUSH, SW27 SW_PUSH, SW28 SW_PUSH, SW29 SW_PUSH, SW3 SW_PUSH, SW30 SW_PUSH, SW31 SW_PUSH, SW32 SW_PUSH, SW33 SW_PUSH, SW34 SW_PUSH, SW35 SW_PUSH, SW36 SW_PUSH, SW37 SW_PUSH, SW38 SW_PUSH, SW39 SW_PUSH, SW4 SW_PUSH, SW5 SW_PUSH, SW6 SW_PUSH, SW7 SW_PUSH, SW8 SW_PUSH, SW9 SW_PUSH, U0 ATmega32U4-AU, U1 PMW3360DM-T2QU, U2 TLV70019DDCR, U3 74LVC1T45GW,125, U4 74LVC1T45GW,125, U5 74LVC1T45GW,125, U6 74LVC1T45GW,125, U7 74LVC1T45GW,125, Y0 16Mhz

Commit message: wip
Connections:
- wire segments 278 -> 276
Changed lines of the file:
@@
 Text GLabel 3050 1150 2    50   Input ~ 0
 SCLK-H
-Connection ~ 2350 4350
 $Comp
 L power:GND #PWR0107
@@
 	1    0    0    -1
 $EndComp
-Wire Wire Line
-	2350 4350 2450 4350
 Text GLabel 1850 1050 0    50   Input ~ 0
 RESET
@@
 $EndComp
 $Comp
-L MCU_Microchip_ATmega:ATmega32U4-AU U0
-U 1 1 60D2737F
-P 2450 2550
-F 0 "U0" H 2625 775 50  0000 C CNN
-F 1 "ATmega32U4-AU" H 2775 700 50  0000 C CNN
-F 2 "Package_QFP:TQFP-44_10x10mm_P0.8mm" H 2450 2550 50  0001 C CIN
-F 3 "http://ww1.microchip.com/downloads/en/DeviceDoc/Atmel-7766-8-bit-AVR-ATmega16U4-32U4_Datasheet.pdf" H 2450 2550 50  0001 C CNN
-	1    2450 2550
-	1    0    0    -1
-$EndComp
-$Comp
 L Device:C C0
 U 1 1 60D2ED48
@@
 	1    0    0    -1
 $EndComp
-Wire Wire Line
-	2350 750  2450 750
 Connection ~ 2450 750
-Wire Wire Line
-	2450 750  2550 750
 $Comp
 L power:VCC #PWR0110
@@
 Text GLabel 10850 2050 0    50   Input ~ 0
 SS-H
+Text GLabel 3050 2950 2    50   Input ~ 0
+col2
+Text GLabel 3050 1550 2    50   Input ~ 0
+col0
 Text GLabel 3050 1450 2    50   Input ~ 0
-row0
-Text GLabel 3050 1550 2    50   Input ~ 0
-row1
-Text GLabel 3050 1650 2    50   Input ~ 0
-row2
+col1
 Text GLabel 3050 1750 2    50   Input ~ 0
 row3
 Text GLabel 3050 2250 2    50   Input ~ 0
-col0
-Text GLabel 3050 2350 2    50   Input ~ 0
-col1
+row2
 Text GLabel 3050 2650 2    50   Input ~ 0
-col2
+col4
 Text GLabel 3050 2750 2    50   Input ~ 0
+row0
+Text GLabel 3050 2850 2    50   Input ~ 0
 col3
-Text GLabel 3050 2850 2    50   Input ~ 0
-col4
-Text GLabel 3050 2950 2    50   Input ~ 0
+Text GLabel 3050 3850 2    50   Input ~ 0
+col9
+Text GLabel 3050 3450 2    50   Input ~ 0
 col5
-Text GLabel 3050 3450 2    50   Input ~ 0
+Text GLabel 3050 3550 2    50   Input ~ 0
 col6
-Text GLabel 3050 3550 2    50   Input ~ 0
+Text GLabel 3050 3650 2    50   Input ~ 0
 col7
-Text GLabel 3050 3650 2    50   Input ~ 0
+Text GLabel 3050 3750 2    50   Input ~ 0
 col8
-Text GLabel 3050 3750 2    50   Input ~ 0
-col9
 NoConn ~ 4725 2400
 NoConn ~ 3050 1950
 NoConn ~ 3050 2050
 NoConn ~ 3050 3950
-NoConn ~ 3050 3850
 NoConn ~ 3050 3250
 NoConn ~ 1850 1650
@@
 Connection ~ 1300 1450
 Wire Wire Line
-	1300 1450 1850 1450
-Connection ~ 1850 1450
-Wire Wire Line
-	1850 1450 1875 1450
-Wire Wire Line
 	1000 1150 1300 1150
 Connection ~ 1300 1150
@@
 Connection ~ 4025 7500
 Wire Wire Line
-	2900 4700 2900 5300
-Wire Wire Line
 	1825 7500 2900 7500
 Connection ~ 2900 7500
@@
 Wire Wire Line
 	3500 4825 3500 5300
-Connection ~ 2900 5300
 Connection ~ 3500 5300
 Wire Wire Line
@@
 Wire Wire Line
 	1825 5900 1825 6500
+Connection ~ 2350 4350
+Wire Wire Line
+	2450 750  2550 750
+Wire Wire Line
+	2350 4350 2450 4350
+Wire Wire Line
+	2350 750  2450 750
+$Comp
+L MCU_Microchip_ATmega:ATmega32U4-AU U0
+U 1 1 60D2737F
+P 2450 2550
+F 0 "U0" H 2625 775 50  0000 C CNN
+F 1 "ATmega32U4-AU" H 2775 700 50  0000 C CNN
+F 2 "Package_QFP:TQFP-44_10x10mm_P0.8mm" H 2450 2550 50  0001 C CIN
+F 3 "http://ww1.microchip.com/downloads/en/DeviceDoc/Atmel-7766-8-bit-AVR-ATmega16U4-32U4_Datasheet.pdf" H 2450 2550 50  0001 C CNN
+	1    2450 2550
+	1    0    0    -1
+$EndComp
+Wire Wire Line
+	1300 1450 1850 1450
+Text GLabel 3050 2350 2    50   Input ~ 0
+row1
+NoConn ~ 3050 1650
 $EndSCHEMATC

Commit message: wip
Parts:
- removed D40, D41, D42, D43, D44, D45: WS2812B, LED_SMD:LED_WS2812B_PLCC4_5.0x5.0mm_P3.2mm, symbol LED:WS2812B
- removed RESET_SW0: SW_PUSH, Keebio-Parts:SW_Tactile_SPST_Angled_MJTP1117, symbol molecule_v2-rescue:SW_PUSH-kbd
- added R8: 10k, Resistor_SMD:R_1206_3216Metric, symbol Device:R
- added RESET_SW0: TS-1187A-B-A-B, TS-1187A-B-A-B:SW_TS-1187A-B-A-B, symbol TS-1187A-B-A-B:TS-1187A-B-A-B
- C7: value 0.1μF -> 4.7μF
- C8: value 4.7μF -> 0.1μF
- LED0, LED1, LED10, LED11, LED12, LED13, LED14, LED15, LED16, LED17, LED18, LED19, LED2, LED20, LED21, LED22, LED23, LED24, LED25, LED26, LED27, LED28, LED29, LED3, LED30, LED31, LED32, LED33, LED34, LED35, LED36, LED37, LED38, LED39, LED4, LED5, LED6, LED7, LED8, LED9: symbol molecule_v2-rescue:YS-SK6812MINI-E-kbd -> kbd:YS-SK6812MINI-E
- SW0, SW1, SW10, SW11, SW12, SW13, SW14, SW15, SW16, SW17, SW18, SW19, SW2, SW20, SW21, SW22, SW23, SW24, SW25, SW26, SW27, SW28, SW29, SW3, SW30, SW31, SW32, SW33, SW34, SW35, SW36, SW37, SW38, SW39, SW4, SW5, SW6, SW7, SW8, SW9: symbol molecule_v2-rescue:SW_PUSH-kbd -> kbd:SW_PUSH
- U1: symbol molecule_v2-rescue:PMW3360DM-T2QU-PMW3360DM-T2QU -> PMW3360DM-T2QU:PMW3360DM-T2QU
- U2: symbol molecule_v2-rescue:TLV70019DDCR-TLV70019DDCR -> TLV70019DDCR:TLV70019DDCR
- U3, U4, U5, U6, U7: symbol molecule_v2-rescue:74LVC1T45GW,125-eec -> 74LVC1T45GW:74LVC1T45GW,125
Connections:
- net labels added: VDD
- wire segments 276 -> 253
- no-connect marks 16 -> 15
