File: hagoromo/hagoromo.kicad_pcb (KiCad board)
At the start: 2 copper layers, 358.9 x 133.9 mm, 189 parts, among them J0 USB_C_Receptacle_USB2.0, SW00_00 SW_PUSH, SW00_11 SW_PUSH, SW01_00 SW_PUSH, SW01_01 SW_PUSH, SW01_02 SW_PUSH, SW01_03 SW_PUSH, SW01_04 SW_PUSH, SW01_05 SW_PUSH, SW01_06 SW_PUSH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

Commit message: kicad version up to 6
Other:
- net class Default removed
