File: dynamis/dynamis.kicad_sch (KiCad schematic)
At the start: 0 parts

Commit message: dynamis render
Parts:
- added C0, C10, C9: 1μF, Capacitor_SMD:C_1206_3216Metric, symbol Device:C
- added C1, C2, C3, C8: 0.1μF, Capacitor_SMD:C_1206_3216Metric, symbol Device:C
- added C4: 10μF, Capacitor_SMD:C_1206_3216Metric, symbol Device:C
- added C5, C6: 22pF, Capacitor_SMD:C_1206_3216Metric, symbol Device:C
- added C7: 4.7μF, Capacitor_SMD:C_1206_3216Metric, symbol Device:C
- added D00_00, D00_01, D00_02, D00_03, D00_04, D00_05, D00_06, D01_00, D01_01, D01_02, D01_03, D01_04, D01_05, D01_06, D02_00, D02_01, D02_02, D02_03, D02_04, D02_05, D02_06, D03_00, D03_01, D03_02, D03_03, D03_04, D03_05, D03_06, D04_00, D04_01, D04_02, D04_03, D04_04, D04_05, D04_06, D05_00, D05_01, D05_02, D05_03, D05_04, D05_05, D05_06, D06_00, D06_01, D06_02, D06_03, D06_04, D06_05, D06_06, D07_00, D07_01, D07_02, D07_03, D07_04, D07_05, D07_06, D08_00, D08_01, D08_02, D08_03, D08_04, D08_05, D08_06, D09_00, D09_01, D09_02, D09_03, D09_04, D09_05, D09_06: D, kbd:D3_SMD_v2, symbol Device:D
- added J0: USB_C_Receptacle_USB2.0, Connector_USB:USB_C_Receptacle_HRO_TYPE-C-31-M-12, symbol Connector:USB_C_Receptacle_USB2.0
- added JP0: SJ, Jumper:SolderJumper-2_P1.3mm_Open_Pad1.0x1.5mm, symbol Jumper:SolderJumper_2_Open
- added LED00, LED01, LED02, LED03, LED04, LED05, LED06, LED07, LED08, LED09: WS2812B, LED_SMD:LED_WS2812B_PLCC4_5.0x5.0mm_P3.2mm, symbol LED:WS2812B
- added R0, R1: 22, Resistor_SMD:R_1206_3216Metric, symbol Device:R
- added R2, R3: 5.1k, Resistor_SMD:R_1206_3216Metric, symbol Device:R
- added R4, R6, R7, R8: 10k, Resistor_SMD:R_1206_3216Metric, symbol Device:R
- added R5: 39, Resistor_SMD:R_1206_3216Metric, symbol Device:R
- added RE0: RotaryEncoder, Rotary_Encoder:RotaryEncoder_Alps_EC12E_Vertical_H20mm, symbol Device:RotaryEncoder
- added RESET_SW0: TS-1187A-B-A-B, TS-1187A-B-A-B:SW_TS-1187A-B-A-B, symbol TS-1187A-B-A-B:TS-1187A-B-A-B
- added SW00_00, SW00_01, SW00_02, SW00_03, SW00_04, SW00_05, SW00_06, SW01_00, SW01_01, SW01_02, SW01_03, SW01_04, SW01_05, SW01_06, SW02_01, SW02_02, SW02_03, SW02_04, SW02_05, SW02_06, SW03_00, SW03_02, SW03_03, SW03_04, SW03_05, SW03_06, SW04_00, SW04_01, SW04_02, SW04_03, SW04_05, SW04_06, SW05_01, SW05_02, SW05_03, SW05_04, SW05_05, SW05_06, SW06_00, SW06_01, SW06_02, SW06_03, SW06_04, SW06_05, SW06_06, SW07_01, SW07_02, SW07_03, SW07_04, SW07_05, SW07_06, SW08_00, SW08_02, SW08_03, SW08_04, SW08_05, SW08_06, SW09_00, SW09_01, SW09_02, SW09_03, SW09_04, SW09_05, SW09_06, SWBS_L00, SWBS_S00, SWCL_N00, SWCL_S00, SWET_AN00, SWET_IS00, SWLS_L00, SWLS_S00, SWRS_L00, SWRS_S00, SWSP_L00, SWSP_S00: SW_Push, kbd:CherryMX_Hotswap, symbol Switch:SW_Push
- added U0: ATmega32U4-A, Package_QFP:TQFP-44_10x10mm_P0.8mm, symbol MCU_Microchip_ATmega:ATmega32U4-A
- added U1: PMW3360DM-T2QU, PMW3360DM-T2QU:PMW3360, symbol PMW3360DM-T2QU:PMW3360DM-T2QU
- added U2: TLV70019DDCR, TLV70019DDCR:Texas_Instruments-TLV70019DDCR-Level_A, symbol TLV70019DDCR:TLV70019DDCR
- added U3, U4, U5, U6, U7: 74LVC1T45GW,125, 74LVC1T45GW:Nexperia-SOT363-11_2018-0-IPC_A, symbol 74LVC1T45GW:74LVC1T45GW,125
- added Y0: 16Mhz, Crystal:Crystal_SMD_SeikoEpson_FA238-4Pin_3.2x2.5mm, symbol Device:Crystal_GND24
Connections:
- new net: R0.1, U0.4 (D+)
- new net: R1.1, U0.3 (D-)
- new net: C0.1, U0.6 (UCAP)
- new net: C7.2, C8.2, U1.3 (VDDPIX)
- new net: R5.2, U1.15 (LED_P)
- new net: JP0.2 (B), R6.2
- new net: J0.A5 (CC1), R2.2
- new net: J0.B5 (CC2), R3.2
- new net: C5.2, U0.17 (XTAL1), Y0.3
- new net: C6.1, U0.16 (XTAL2), Y0.1
- new net: R8.1, U1.7 (NRESET)
- new net: R7.2, U0.33 (~{HWB}/PE2)
- new net: D02_02.2 (A), SW02_02.2
- new net: D07_03.2 (A), SW07_03.2
- new net: D04_06.2 (A), SW04_06.2
- new net: D07_04.2 (A), SW07_04.2
- new net: D06_01.2 (A), SW06_01.2
- new net: D08_01.2 (A), SWRS_L00.2, SWRS_S00.2
- new net: D03_03.2 (A), SW03_03.2
- new net: D09_05.2 (A), SW09_05.2
- new net: D01_01.2 (A), SW01_01.2
- new net: D03_02.2 (A), SW03_02.2
- new net: D01_05.2 (A), SW01_05.2
- new net: LED07.2 (DOUT), LED08.4 (DIN)
- new net: LED06.2 (DOUT), LED07.4 (DIN)
- new net: D04_00.2 (A), SW04_00.2
- new net: D06_02.2 (A), SW06_02.2
- new net: D09_01.2 (A), SW09_01.2
- new net: D08_02.2 (A), SW08_02.2
- new net: D01_06.2 (A), SW01_06.2
- new net: D06_06.2 (A), SW06_06.2
- new net: D07_00.2 (A), SWET_AN00.2, SWET_IS00.2
- new net: D00_03.2 (A), SW00_03.2
- new net: D00_00.2 (A), SW00_00.2
- new net: D06_03.2 (A), SW06_03.2
- new net: D05_01.2 (A), SW05_01.2
- new net: D05_04.2 (A), SW05_04.2
- new net: D08_00.2 (A), SW08_00.2
- new net: D05_00.2 (A), SWBS_L00.2, SWBS_S00.2
- new net: D04_04.2 (A), SWSP_L00.2, SWSP_S00.2
- new net: D09_04.2 (A), SW09_04.2
- new net: D07_05.2 (A), SW07_05.2
- new net: D08_04.2 (A), SW08_04.2
- new net: D05_03.2 (A), SW05_03.2
- new net: D03_06.2 (A), SW03_06.2
- new net: D05_05.2 (A), SW05_05.2
- new net: D02_04.2 (A), SW02_04.2
- new net: D02_03.2 (A), SW02_03.2
- new net: D04_01.2 (A), SW04_01.2
- new net: D03_04.2 (A), SW03_04.2
- new net: LED05.2 (DOUT), LED06.4 (DIN)
- new net: LED08.2 (DOUT), LED09.4 (DIN)
- new net: D04_05.2 (A), SW04_05.2
- new net: D06_05.2 (A), SW06_05.2
- new net: D02_06.2 (A), SW02_06.2
- new net: D08_05.2 (A), SW08_05.2
- new net: D02_05.2 (A), SW02_05.2
- new net: D04_02.2 (A), SW04_02.2
- new net: D01_04.2 (A), SW01_04.2
- new net: D00_02.2 (A), SW00_02.2
- new net: D09_02.2 (A), SW09_02.2
- new net: D03_01.2 (A), SWLS_L00.2, SWLS_S00.2
- new net: D05_02.2 (A), SW05_02.2
- new net: D03_05.2 (A), SW03_05.2
- new net: D08_06.2 (A), SW08_06.2
- new net: LED04.2 (DOUT), LED05.4 (DIN)
- new net: D07_01.2 (A), SW07_01.2
- new net: D03_00.2 (A), SW03_00.2
- new net: D09_06.2 (A), SW09_06.2
- new net: D06_04.2 (A), SW06_04.2
- new net: D09_03.2 (A), SW09_03.2
- new net: D00_06.2 (A), SW00_06.2
- new net: LED02.2 (DOUT), LED03.4 (DIN)
- new net: LED01.2 (DOUT), LED02.4 (DIN)
- new net: D00_01.2 (A), SW00_01.2
- new net: D06_00.2 (A), SW06_00.2
- new net: D01_02.2 (A), SW01_02.2
- new net: D01_03.2 (A), SW01_03.2
- new net: D05_06.2 (A), SW05_06.2
- new net: D02_00.2 (A), SWCL_N00.2, SWCL_S00.2
- new net: LED03.2 (DOUT), LED04.4 (DIN)
- new net: D01_00.2 (A), SW01_00.2
- new net: D00_04.2 (A), SW00_04.2
- new net: D08_03.2 (A), SW08_03.2
- new net: D00_05.2 (A), SW00_05.2
- new net: D07_06.2 (A), SW07_06.2
- new net: LED00.2 (DOUT), LED01.4 (DIN)
- new net: D07_02.2 (A), SW07_02.2
- new net: D04_03.2 (A), SW04_03.2
- new net: D02_01.2 (A), SW02_01.2
- new net: D09_00.2 (A), SW09_00.2
- new net D+: J0.A6 (D+), J0.B6 (D+), R0.2
- new net D-: J0.A7 (D-), J0.B7 (D-), R1.2
- new net GND: C0.2, C1.2, C10.2, C2.2, C3.2, C4.2, C5.1, C6.2, C7.1, C8.1, C9.2, J0.A1 (GND), J0.A12 (GND), J0.B1 (GND), J0.B12 (GND), J0.S1 (SHIELD), LED00.3 (VSS), LED01.3 (VSS), LED02.3 (VSS), LED03.3 (VSS), LED04.3 (VSS), LED05.3 (VSS), LED06.3 (VSS), LED07.3 (VSS), LED08.3 (VSS), LED09.3 (VSS), R2.1, R3.1, R7.1, RE0.C, RESET_SW0.C, RESET_SW0.D, U0.15 (GND), U0.23 (GND), U0.35 (GND), U0.43 (GND), U0.5 (UGND), U1.8 (GND), U2.2 (GND), U3.2 (GND), U4.2 (GND), U5.2 (GND), U6.2 (GND), U6.5 (DIR), U7.2 (GND), Y0.2, Y0.4
- new net LED: LED00.4 (DIN), U0.21 (PD3)
- new net MISO: JP0.1 (A), U1.12 (MISO), U7.4 (B)
- new net MISO-H: U0.11 (PB3), U7.3 (A)
- new net MOSI: U1.11 (MOSI), U3.4 (B)
- new net MOSI-H: U0.10 (PB2), U3.3 (A)
- new net MOT-H: U0.20 (PD2), U6.3 (A)
- new net MOTION: U1.9 (MOTION), U6.4 (B)
- new net RESET: R4.2, RESET_SW0.A, RESET_SW0.B, U0.13 (~{RESET})
- new net RE_A: RE0.A, U0.12 (PB7)
- new net RE_B: RE0.B, U0.1 (PE6)
- new net SCLK: U1.10 (SCLK), U4.4 (B)
- new net SCLK-H: U0.9 (PB1), U4.3 (A)
- new net SS: U1.13 (NCS), U5.4 (B)
- new net SS-H: U0.8 (PB0), U5.3 (A), U7.5 (DIR)
- new net VCC: C1.1, C10.1, C2.1, C3.1, C4.1, J0.A4 (VBUS), J0.A9 (VBUS), J0.B4 (VBUS), J0.B9 (VBUS), LED00.1 (VDD), LED01.1 (VDD), LED02.1 (VDD), LED03.1 (VDD), LED04.1 (VDD), LED05.1 (VDD), LED06.1 (VDD), LED07.1 (VDD), LED08.1 (VDD), LED09.1 (VDD), R4.1, U0.14 (VCC), U0.2 (UVCC), U0.24 (AVCC), U0.34 (VCC), U0.44 (AVCC), U0.7 (VBUS), U2.1 (IN), U2.3 (EN), U3.1 (VCC(A)), U3.5 (DIR), U4.1 (VCC(A)), U4.5 (DIR), U5.1 (VCC(A)), U5.5 (DIR), U6.1 (VCC(A)), U7.1 (VCC(A))
- new net VDD: C9.1, R5.1, R6.1, R8.2, U1.4 (VDD), U1.5 (VDDIO), U2.5 (OUT), U3.6 (VCC(B)), U4.6 (VCC(B)), U5.6 (VCC(B)), U6.6 (VCC(B)), U7.6 (VCC(B))
- new net col00: SW00_00.1, SW01_00.1, SW03_00.1, SW04_00.1, SW06_00.1, SW08_00.1, SW09_00.1, SWBS_L00.1, SWBS_S00.1, SWCL_N00.1, SWCL_S00.1, SWET_AN00.1, SWET_IS00.1, U0.41 (PF0)
- new net col01: SW00_01.1, SW01_01.1, SW02_01.1, SW04_01.1, SW05_01.1, SW06_01.1, SW07_01.1, SW09_01.1, SWLS_L00.1, SWLS_S00.1, SWRS_L00.1, SWRS_S00.1, U0.40 (PF1)
- new net col02: SW00_02.1, SW01_02.1, SW02_02.1, SW03_02.1, SW04_02.1, SW05_02.1, SW06_02.1, SW07_02.1, SW08_02.1, SW09_02.1, U0.39 (PF4)
- new net col03: SW00_03.1, SW01_03.1, SW02_03.1, SW03_03.1, SW04_03.1, SW05_03.1, SW06_03.1, SW07_03.1, SW08_03.1, SW09_03.1, U0.38 (PF5)
- new net col04: SW00_04.1, SW01_04.1, SW02_04.1, SW03_04.1, SW05_04.1, SW06_04.1, SW07_04.1, SW08_04.1, SW09_04.1, SWSP_L00.1, SWSP_S00.1, U0.37 (PF6)
- new net col05: SW00_05.1, SW01_05.1, SW02_05.1, SW03_05.1, SW04_05.1, SW05_05.1, SW06_05.1, SW07_05.1, SW08_05.1, SW09_05.1, U0.36 (PF7)
- new net col06: SW00_06.1, SW01_06.1, SW02_06.1, SW03_06.1, SW04_06.1, SW05_06.1, SW06_06.1, SW07_06.1, SW08_06.1, SW09_06.1, U0.32 (PC7)
- new net row00: D00_00.1 (K), D00_01.1 (K), D00_02.1 (K), D00_03.1 (K), D00_04.1 (K), D00_05.1 (K), D00_06.1 (K), U0.30 (PB6)
- new net row01: D01_00.1 (K), D01_01.1 (K), D01_02.1 (K), D01_03.1 (K), D01_04.1 (K), D01_05.1 (K), D01_06.1 (K), U0.28 (PB4)
- new net row02: D02_00.1 (K), D02_01.1 (K), D02_02.1 (K), D02_03.1 (K), D02_04.1 (K), D02_05.1 (K), D02_06.1 (K), U0.26 (PD6)
- new net row03: D03_00.1 (K), D03_01.1 (K), D03_02.1 (K), D03_03.1 (K), D03_04.1 (K), D03_05.1 (K), D03_06.1 (K), U0.22 (PD5)
- new net row04: D04_00.1 (K), D04_01.1 (K), D04_02.1 (K), D04_03.1 (K), D04_04.1 (K), D04_05.1 (K), D04_06.1 (K), U0.19 (PD1)
- new net row05: D05_00.1 (K), D05_01.1 (K), D05_02.1 (K), D05_03.1 (K), D05_04.1 (K), D05_05.1 (K), D05_06.1 (K), U0.31 (PC6)
- new net row06: D06_00.1 (K), D06_01.1 (K), D06_02.1 (K), D06_03.1 (K), D06_04.1 (K), D06_05.1 (K), D06_06.1 (K), U0.29 (PB5)
- new net row07: D07_00.1 (K), D07_01.1 (K), D07_02.1 (K), D07_03.1 (K), D07_04.1 (K), D07_05.1 (K), D07_06.1 (K), U0.27 (PD7)
- new net row08: D08_00.1 (K), D08_01.1 (K), D08_02.1 (K), D08_03.1 (K), D08_04.1 (K), D08_05.1 (K), D08_06.1 (K), U0.25 (PD4)
- new net row09: D09_00.1 (K), D09_01.1 (K), D09_02.1 (K), D09_03.1 (K), D09_04.1 (K), D09_05.1 (K), D09_06.1 (K), U0.18 (PD0)
- no-connect marks 0 -> 10
Other:
- title: (none) -> hogoromo
