File: dynamis/case/plate/dynamis-plate.kicad_pcb (KiCad board)
At the start: 2 copper layers, 339.9 x 106.6 mm, 0 parts

Commit message: dynamis render
Parts:
- added LOGO: LOGO, dynamis:logo, F.Cu at (356.4, 104.9)
Other:
- outline, holes or cut-outs redrawn
- board text added: "dynamis v1.0.0 designed by bbrfkr"

Commit message: mod plate
Other:
- outline, holes or cut-outs redrawn
