File: dynamis/case/sandwitch/dynamis-sandwitch.kicad_pcb (KiCad board)
At the start: 2 copper layers, 339.9 x 106.6 mm, 0 parts

Commit message: mod plate
Parts:
- added LOGO01: LOGO, dynamis:logo, B.Cu at (371.8, 187.4)
Changed lines of the file:
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@@
   )
   (net 0 "")
+  (footprint "dynamis:logo" (layer "B.Cu")
+    (at 371.7544 187.3758 180)
+    (attr board_only exclude_from_pos_files exclude_from_bom)
+    (fp_text reference "LOGO01" (at 0 0) (layer "Cmts.User")
+      (effects (font (size 1.524 1.524) (thickness 0.3)))
+    )
+    (fp_text value "LOGO" (at 0.75 0) (layer "Cmts.User") hide
+      (effects (font (size 1.524 1.524) (thickness 0.3)))
+    )
+    (fp_poly (pts
+        (xy 1.164129 4.723378)
+        (xy 2.226658 3.048001)
+        (xy 1.214929 3.048001)
+        (xy 0.636606 3.025653)
+        (xy 0.270413 2.96854)
+        (xy 0.2032 2.924326)
+        (xy 0.315302 2.713666)
+        (xy 0.613014 2.264056)
+        (xy 1.038444 1.661919)
+        (xy 1.1684 1.483445)
+        (xy 2.1336 0.166239)
+        (xy 2.2352 1.54004)
+        (xy 2.3368 2.913842)
+        (xy 3.298454 1.464689)
+        (xy 4.260108 0.015535)
+        (xy 2.227416 -3.091032)
+        (xy 1.570981 -4.083569)
+        (xy 0.983694 -4.951405)
+        (xy 0.503848 -5.639569)
+        (xy 0.169735 -6.093088)
+        (xy 0.022472 -6.256429)
+        (xy -0.137612 -6.113316)
+        (xy -0.477935 -5.679856)
+        (xy -0.960642 -5.008622)
+        (xy -1.547875 -4.152188)
+        (xy -2.172309 -3.208429)
+        (xy -4.168152 -0.142593)
+        (xy -2.2352 -0.142593)
+        (xy -2.2352 -3.048)
+        (xy -1.2192 -3.048)
+        (xy -0.639459 -3.028093)
+        (xy -0.271611 -2.977197)
+        (xy -0.2032 -2.937401)
+        (xy -0.317611 -2.735436)
+        (xy -0.622136 -2.294657)
+        (xy -1.058719 -1.698077)
+        (xy -1.2192 -1.484698)
+        (xy -2.2352 -0.142593)
+        (xy -4.168152 -0.142593)
+        (xy -4.194838 -0.1016)
+        (xy -3.199356 -0.039637)
+        (xy -2.203874 0.022325)
+        (xy -2.208325 0.123675)
+        (xy -2.032 0.123675)
+        (xy -1.849141 0.053107)
+        (xy -1.381626 0.00833)
+        (xy -1.016 0)
+        (xy 0 0)
+        (xy 0 1.4224)
+        (xy -0.008164 2.123559)
+        (xy -0.029646 2.631594)
+        (xy -0.059937 2.84369)
+        (xy -0.06241 2.8448)
+        (xy -0.209491 2.693186)
+        (xy -0.516872 2.302321)
+        (xy -0.91509 1.76817)
+        (xy -1.334684 1.186702)
+        (xy -1.70619 0.653881)
+        (xy -1.960148 0.265676)
+        (xy -2.032 0.123675)
+        (xy -2.208325 0.123675)
+        (xy -2.270337 1.535636)
+        (xy -2.3368 3.048946)
+        (xy -1.176618 3.048473)
+        (xy -0.016436 3.048001)
+        (xy 0.042582 4.723378)
+        (xy 0.1016 6.398756)
+      ) (layer "B.Mask") (width 0) (fill solid))
+  )
   (gr_line (start 329.844982 153.451394) (end 329.487988 153.212895) (layer "Edge.Cuts") (width 0.1))
   (gr_line (start 42.079414 194.5239) (end 42.079414 194.5239) (layer "Edge.Cuts") (width 0.1))
@@
   (gr_line (start 251.266018 135.547394) (end 250.910015 135.308995) (layer "Edge.Cuts") (width 0.1))
   (gr_line (start 376.350018 93.54005) (end 376.682995 93.31503) (layer "Edge.Cuts") (width 0.1))
-  (gr_text "dynamis v1.0.0 designed by bbrfkr" (at 354.33 192.786) (layer "B.Mask")
-    (effects (font (size 1.5 1.5) (thickness 0.3)) (justify mirror))
+  (gr_text "dynamis v1.0.0 designed by bbrfkr" (at 354.33 192.786) (layer "F.Mask")
+    (effects (font (size 1.5 1.5) (thickness 0.3)))
   )
   (zone (net 0) (net_name "") (layer "F.Cu") (hatch edge 0.508)
